File: rgb_matrix.kicad_sch (KiCad schematic)
At the start: 0 parts

Commit message: added rgb matrix
Parts:
- added C11 (x29): 0.1µ, symbol Device:C
- added D32, D33, D34, D35, D36, D37, D38, D39, D40, D41, D42, D43, D44, D45, D46, D47, D48, D49, D50, D51, D52, D53, D54, D55, D56, D57, D58, D59, D60: SK6812MINI, LED_SMD:LED_SK6812MINI_PLCC4_3.5x3.5mm_P1.75mm, symbol LED:SK6812MINI
- added R11: 540, symbol Device:R
Connections:
- new net: D50.1 (DOUT), D51.3 (DIN)
- new net: D49.1 (DOUT), D50.3 (DIN)
- new net: D54.1 (DOUT), D55.3 (DIN)
- new net: D53.1 (DOUT), D54.3 (DIN)
- new net: D48.1 (DOUT), D49.3 (DIN)
- new net: D47.1 (DOUT), D48.3 (DIN)
- new net: D51.1 (DOUT), D52.3 (DIN)
- new net: D52.1 (DOUT), D53.3 (DIN)
- new net: D59.1 (DOUT), D60.3 (DIN)
- new net: D43.1 (DOUT), D44.3 (DIN)
- new net: D42.1 (DOUT), D43.3 (DIN)
- new net: D45.1 (DOUT), D46.3 (DIN)
- new net: D44.1 (DOUT), D45.3 (DIN)
- new net: D58.1 (DOUT), D59.3 (DIN)
- new net: D57.1 (DOUT), D58.3 (DIN)
- new net: D39.1 (DOUT), D40.3 (DIN)
- new net: D38.1 (DOUT), D39.3 (DIN)
- new net: D37.1 (DOUT), D38.3 (DIN)
- new net: D32.3 (DIN), R11.2
- new net: D41.1 (DOUT), D42.3 (DIN)
- new net: D40.1 (DOUT), D41.3 (DIN)
- new net: D46.1 (DOUT), D47.3 (DIN)
- new net: D32.1 (DOUT), D33.3 (DIN)
- new net: D33.1 (DOUT), D34.3 (DIN)
- new net: D35.1 (DOUT), D36.3 (DIN)
- new net: D34.1 (DOUT), D35.3 (DIN)
- new net: D36.1 (DOUT), D37.3 (DIN)
- new net: D56.1 (DOUT), D57.3 (DIN)
- new net: D55.1 (DOUT), D56.3 (DIN)
- new net +5V: C11.1, C11.1, C11.1, C11.1, C11.1, C11.1, C11.1, C11.1, C11.1, C11.1, C11.1, C11.1, C11.1, C11.1, C11.1, C11.1, C11.1, C11.1, C11.1, C11.1, C11.1, C11.1, C11.1, C11.1, C11.1, C11.1, C11.1, C11.1, C11.1, D32.4 (VDD), D33.4 (VDD), D34.4 (VDD), D35.4 (VDD), D36.4 (VDD), D37.4 (VDD), D38.4 (VDD), D39.4 (VDD), D40.4 (VDD), D41.4 (VDD), D42.4 (VDD), D43.4 (VDD), D44.4 (VDD), D45.4 (VDD), D46.4 (VDD), D47.4 (VDD), D48.4 (VDD), D49.4 (VDD), D50.4 (VDD), D51.4 (VDD), D52.4 (VDD), D53.4 (VDD), D54.4 (VDD), D55.4 (VDD), D56.4 (VDD), D57.4 (VDD), D58.4 (VDD), D59.4 (VDD), D60.4 (VDD)
- new net GND: C11.2, C11.2, C11.2, C11.2, C11.2, C11.2, C11.2, C11.2, C11.2, C11.2, C11.2, C11.2, C11.2, C11.2, C11.2, C11.2, C11.2, C11.2, C11.2, C11.2, C11.2, C11.2, C11.2, C11.2, C11.2, C11.2, C11.2, C11.2, C11.2, D32.2 (VSS), D33.2 (VSS), D34.2 (VSS), D35.2 (VSS), D36.2 (VSS), D37.2 (VSS), D38.2 (VSS), D39.2 (VSS), D40.2 (VSS), D41.2 (VSS), D42.2 (VSS), D43.2 (VSS), D44.2 (VSS), D45.2 (VSS), D46.2 (VSS), D47.2 (VSS), D48.2 (VSS), D49.2 (VSS), D50.2 (VSS), D51.2 (VSS), D52.2 (VSS), D53.2 (VSS), D54.2 (VSS), D55.2 (VSS), D56.2 (VSS), D57.2 (VSS), D58.2 (VSS), D59.2 (VSS), D60.2 (VSS)
- new net RGB_data: R11.1

Commit message: added power switch for rgb
Connections:
- net +5V renamed VCC
Changed lines of the file:
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@@
     (stroke (width 0) (type default))
+  )
+  (hierarchical_label "VCC" (shape input) (at 29.21 53.34 180) (fields_autoplaced)
+    (effects (font (size 1.27 1.27)) (justify right))
+  )
+  (hierarchical_label "VCC" (shape input) (at 29.21 16.51 180) (fields_autoplaced)
+    (effects (font (size 1.27 1.27)) (justify right))
+  )
+  (hierarchical_label "VCC" (shape input) (at 29.21 90.17 180) (fields_autoplaced)
+    (effects (font (size 1.27 1.27)) (justify right))
+  )
+  (hierarchical_label "VCC" (shape input) (at 29.21 163.83 180) (fields_autoplaced)
+    (effects (font (size 1.27 1.27)) (justify right))
+  )
+  (hierarchical_label "VCC" (shape input) (at 29.21 127 180) (fields_autoplaced)
+    (effects (font (size 1.27 1.27)) (justify right))
   )
   (hierarchical_label "RGB_data" (shape input) (at 25.4 35.56 180) (fields_autoplaced)
@@
     )
   )
-  (symbol (lib_id "power:+5V") (at 29.21 127 90) (unit 1)
-    (in_bom yes) (on_board yes) (dnp no) (fields_autoplaced)
-    (property "Reference" "#PWR028" (at 33.02 127 0)
-      (effects (font (size 1.27 1.27)) hide)
-    )
-    (property "Value" "+5V" (at 25.4 127 90)
-      (effects (font (size 1.27 1.27)) (justify left))
-    )
-    (property "Footprint" "" (at 29.21 127 0)
-      (effects (font (size 1.27 1.27)) hide)
-    )
-    (property "Datasheet" "" (at 29.21 127 0)
-      (effects (font (size 1.27 1.27)) hide)
-    )
-    (pin "1")
-    (instances
-      (project "Lily58"
-        (path "/a0958e12-2248-4ac3-b259-3086ac296b70"
-          (reference "#PWR028") (unit 1)
-        )
-        (path "/a0958e12-2248-4ac3-b259-3086ac296b70/3cabbf22-a691-4141-b2a0-7c2cb7676c85"
-          (reference "#PWR080") (unit 1)
-        )
-      )
-    )
-  )
   (symbol (lib_id "Device:C") (at 36.83 57.15 0) (unit 1)
     (in_bom yes) (on_board yes) (dnp no)
@@
     )
   )
-  (symbol (lib_id "power:+5V") (at 29.21 163.83 90) (unit 1)
-    (in_bom yes) (on_board yes) (dnp no) (fields_autoplaced)
-    (property "Reference" "#PWR028" (at 33.02 163.83 0)
-      (effects (font (size 1.27 1.27)) hide)
-    )
-    (property "Value" "+5V" (at 25.4 163.83 90)
-      (effects (font (size 1.27 1.27)) (justify left))
-    )
-    (property "Footprint" "" (at 29.21 163.83 0)
-      (effects (font (size 1.27 1.27)) hide)
-    )
-    (property "Datasheet" "" (at 29.21 163.83 0)
-      (effects (font (size 1.27 1.27)) hide)
-    )
-    (pin "1")
-    (instances
-      (project "Lily58"
-        (path "/a0958e12-2248-4ac3-b259-3086ac296b70"
-          (reference "#PWR028") (unit 1)
-        )
-        (path "/a0958e12-2248-4ac3-b259-3086ac296b70/3cabbf22-a691-4141-b2a0-7c2cb7676c85"
-          (reference "#PWR093") (unit 1)
-        )
-      )
-    )
-  )
   (symbol (lib_id "Device:C") (at 92.71 167.64 0) (unit 1)
     (in_bom yes) (on_board yes) (dnp no)
@@
     )
   )
-  (symbol (lib_id "power:+5V") (at 29.21 53.34 90) (unit 1)
-    (in_bom yes) (on_board yes) (dnp no) (fields_autoplaced)
-    (property "Reference" "#PWR028" (at 33.02 53.34 0)
-      (effects (font (size 1.27 1.27)) hide)
-    )
-    (property "Value" "+5V" (at 25.4 53.34 90)
-      (effects (font (size 1.27 1.27)) (justify left))
-    )
-    (property "Footprint" "" (at 29.21 53.34 0)
-      (effects (font (size 1.27 1.27)) hide)
-    )
-    (property "Datasheet" "" (at 29.21 53.34 0)
-      (effects (font (size 1.27 1.27)) hide)
-    )
-    (pin "1")
-    (instances
-      (project "Lily58"
-        (path "/a0958e12-2248-4ac3-b259-3086ac296b70"
-          (reference "#PWR028") (unit 1)
-        )
-        (path "/a0958e12-2248-4ac3-b259-3086ac296b70/3cabbf22-a691-4141-b2a0-7c2cb7676c85"
-          (reference "#PWR054") (unit 1)
-        )
-      )
-    )
-  )
   (symbol (lib_id "power:GND") (at 92.71 134.62 0) (unit 1)
     (in_bom yes) (on_board yes) (dnp no) (fields_autoplaced)
@@
     )
   )
-  (symbol (lib_id "power:+5V") (at 29.21 90.17 90) (unit 1)
-    (in_bom yes) (on_board yes) (dnp no) (fields_autoplaced)
-    (property "Reference" "#PWR028" (at 33.02 90.17 0)
-      (effects (font (size 1.27 1.27)) hide)
-    )
-    (property "Value" "+5V" (at 25.4 90.17 90)
-      (effects (font (size 1.27 1.27)) (justify left))
-    )
-    (property "Footprint" "" (at 29.21 90.17 0)
-      (effects (font (size 1.27 1.27)) hide)
-    )
-    (property "Datasheet" "" (at 29.21 90.17 0)
-      (effects (font (size 1.27 1.27)) hide)
-    )
-    (pin "1")
-    (instances
-      (project "Lily58"
-        (path "/a0958e12-2248-4ac3-b259-3086ac296b70"
-          (reference "#PWR028") (unit 1)
-        )
-        (path "/a0958e12-2248-4ac3-b259-3086ac296b70/3cabbf22-a691-4141-b2a0-7c2cb7676c85"
-          (reference "#PWR067") (unit 1)
-        )
-      )
-    )
-  )
   (symbol (lib_id "power:GND") (at 185.42 153.67 0) (unit 1)
     (in_bom yes) (on_board yes) (dnp no) (fields_autoplaced)
@@
         )
       )
-    )
-  )
-  (symbol (lib_id "power:+5V") (at 29.21 16.51 90) (unit 1)
-    (in_bom yes) (on_board yes) (dnp no) (fields_autoplaced)
-    (property "Reference" "#PWR028" (at 33.02 16.51 0)
-      (effects (font (size 1.27 1.27)) hide)
-    )
-    (property "Value" "+5V" (at 25.4 16.51 90)
-      (effects (font (size 1.27 1.27)) (justify left))
-    )
-    (property "Footprint" "" (at 29.21 16.51 0)
-      (effects (font (size 1.27 1.27)) hide)
-    )
-    (property "Datasheet" "" (at 29.21 16.51 0)
-      (effects (font (size 1.27 1.27)) hide)
-    )
-    (pin "1")
-    (instances
-      (project "Lily58"
-        (path "/a0958e12-2248-4ac3-b259-3086ac296b70"
-          (reference "#PWR028") (unit 1)
-        )
-        (path "/a0958e12-2248-4ac3-b259-3086ac296b70/3cabbf22-a691-4141-b2a0-7c2cb7676c85"
-          (reference "#PWR041") (unit 1)
-        )
-      )
